Commit message: feat: Add namespace and switch to gazebo controller

File: pinky_description/urdf/pinky.urdf.xacro (robot description, xacro)
@@ -1,5 +1,5 @@
 <?xml version="1.0"?>
 <robot xmlns:xacro="http://www.ros.org/wiki/xacro">
-    <xacro:macro name="insert_robot" params="namespace is_sim:=false sim_type:=gz_sim cam_tilt_deg screen_tilt_deg">
+    <xacro:macro name="insert_robot" params="namespace is_sim:=false sim_type:=gz_sim ros2_control:=false cam_tilt_deg screen_tilt_deg">
         <xacro:include filename="$(find pinky_description)/urdf/common/insert_inertia.urdf.xacro"/>
         <xacro:include filename="$(find pinky_description)/urdf/pinky_ros2_control.urdf.xacro"/>
@@ -49,5 +49,5 @@
                 </inertial>
             </link>
-            <joint name="${side}_wheel_joint" type="continuous">
+            <joint name="${namespace}${side}_wheel_joint" type="continuous">
                 <parent link="base_link"/>
                 <child link="${side}_wheel"/>
@@ -77,5 +77,5 @@
             </inertial>
         </link>
-        <joint name="caster_mount_fixed_joint" type="fixed">
+        <joint name="${namespace}caster_mount_fixed_joint" type="fixed">
             <parent link="base_link"/>
             <child link="caster_mount_link"/>
@@ -101,5 +101,5 @@
             </inertial>
         </link>
-        <joint name="caster_rotate_joint" type="continuous">
+        <joint name="${namespace}caster_rotate_joint" type="continuous">
             <parent link="caster_mount_link"/>
             <child link="caster_roate_link"/>
@@ -126,5 +126,5 @@
             </inertial>
         </link>
-        <joint name="caster_wheel_joint" type="continuous">
+        <joint name="${namespace}caster_wheel_joint" type="continuous">
             <parent link="caster_roate_link"/>
             <child link="caster_wheel"/>
@@ -151,5 +151,5 @@
             </inertial>
         </link>
-        <joint name="robot_lamp_mount_fixed_joint" type="fixed">
+        <joint name="${namespace}robot_lamp_mount_fixed_joint" type="fixed">
             <parent link="base_link"/>
             <child link="robot_lamp"/>
@@ -175,5 +175,5 @@
             </inertial>
         </link>
-        <joint name="rplidar_mount_fixed_joint" type="fixed">
+        <joint name="${namespace}rplidar_mount_fixed_joint" type="fixed">
             <parent link="base_link"/>
             <child link="rplidar_mount"/>
@@ -181,5 +181,5 @@
         </joint>
         <link name="rplidar_link"/>
-        <joint name="rplidar_link_fixed_joint" type="fixed">
+        <joint name="${namespace}rplidar_link_fixed_joint" type="fixed">
             <parent link="rplidar_mount"/>
             <child link="rplidar_link"/>
@@ -205,5 +205,5 @@
             </inertial>
         </link>
-        <joint name="front_camera_mount_fixed_joint" type="fixed">
+        <joint name="${namespace}front_camera_mount_fixed_joint" type="fixed">
             <parent link="base_link"/>
             <child link="front_camera_mount"/>
@@ -211,5 +211,5 @@
         </joint>
         <link name="front_camera_link"/>
-        <joint name="front_camera_fixed_joint" type="fixed">
+        <joint name="${namespace}front_camera_fixed_joint" type="fixed">
             <parent link="front_camera_mount"/>
             <child link="front_camera_link"/>
@@ -235,5 +235,5 @@
             </inertial>
         </link>
-        <joint name="screen_mount_fixed_joint" type="fixed">
+        <joint name="${namespace}screen_mount_fixed_joint" type="fixed">
             <parent link="base_link"/>
             <child link="screen_mount"/>
@@ -241,5 +241,5 @@
         </joint>
         <link name="ultrasonic_link"/>
-        <joint name="ultrasonic_fixed_joint" type="fixed">
+        <joint name="${namespace}ultrasonic_fixed_joint" type="fixed">
             <parent link="base_link"/>
             <child link="ultrasonic_link"/>
@@ -247,5 +247,5 @@
         </joint>
         <link name="ir_mid_link"/>
-        <joint name="ir_mid_fixed_joint" type="fixed">
+        <joint name="${namespace}ir_mid_fixed_joint" type="fixed">
             <parent link="base_link"/>
             <child link="ir_mid_link"/>
@@ -253,5 +253,5 @@
         </joint>
         <link name="ir_l_link"/>
-        <joint name="ir_l_fixed_joint" type="fixed">
+        <joint name="${namespace}ir_l_fixed_joint" type="fixed">
             <parent link="base_link"/>
             <child link="ir_l_link"/>
@@ -259,5 +259,5 @@
         </joint>
         <link name="ir_r_link"/>
-        <joint name="ir_r_fixed_joint" type="fixed">
+        <joint name="${namespace}ir_r_fixed_joint" type="fixed">
             <parent link="base_link"/>
             <child link="ir_r_link"/>
@@ -265,5 +265,5 @@
         </joint>
         <link name="imu_link"/>
-        <joint name="imu_fixed_joint" type="fixed">
+        <joint name="${namespace}imu_fixed_joint" type="fixed">
             <parent link="base_link"/>
             <child link="imu_link"/>
@@ -273,8 +273,10 @@
             <xacro:if value="${sim_type == 'gz_sim'}">
                 <xacro:include filename="$(find pinky_description)/urdf/pinky_gz.urdf.xacro"/>
-                <xacro:insert_gz_sim namespace="${namespace}"/>
+                <xacro:insert_gz_sim namespace="${namespace}" ros2_control="${ros2_control}"/>
             </xacro:if>
         </xacro:if>
-        <xacro:insert_ros2_control name="pinky" is_sim="${is_sim}" sim_type="${sim_type}"/>
+        <xacro:if value="${ros2_control}">
+            <xacro:insert_ros2_control name="pinky" is_sim="${is_sim}" sim_type="${sim_type}"/>
+        </xacro:if>
     </xacro:macro>
 </robot>

File: pinky_description/urdf/pinky_gz.urdf.xacro (robot description, xacro)
@@ -1,19 +1,44 @@
 <?xml version="1.0"?>
 <robot xmlns:xacro="http://www.ros.org/wiki/xacro">
-    <xacro:macro name="insert_gz_sim" params="namespace">
+    <xacro:macro name="insert_gz_sim" params="namespace ros2_control">
         <gazebo>
-            <plugin filename="gz_ros2_control-system" name="gz_ros2_control::GazeboSimROS2ControlPlugin">
-                <ros>
-                    <namespace>${namespace}</namespace>
-                    <remapping>base_controller/cmd_vel:=cmd_vel</remapping>
-                    <remapping>base_controller/odom:=odom</remapping>
-                </ros>
-                <parameters>$(find pinky_bringup)/config/pinky_controllers.yaml</parameters>
-            </plugin>
+            <xacro:if value="${ros2_control}">
+                <plugin filename="gz_ros2_control-system" name="gz_ros2_control::GazeboSimROS2ControlPlugin">
+                    <ros>
+                        <namespace>${namespace}</namespace>
+                        <remapping>base_controller/cmd_vel:=cmd_vel</remapping>
+                        <remapping>base_controller/odom:=odom</remapping>
+                    </ros>
+                    <parameters>$(find pinky_bringup)/config/pinky_controllers.yaml</parameters>
+                </plugin>
+            </xacro:if>
+            <xacro:unless value="${ros2_control}">
+                <plugin filename="gz-sim-diff-drive-system" name="gz::sim::systems::DiffDrive">
+                    <left_joint>${namespace}l_wheel_joint</left_joint>
+                    <right_joint>${namespace}r_wheel_joint</right_joint>
+                    <wheel_separation>0.0961</wheel_separation>
+                    <wheel_radius>0.028</wheel_radius>
+                    <min_velocity>-1.0</min_velocity>
+                    <max_velocity>1.0</max_velocity>
+                    <min_acceleration>-2.0</min_acceleration>
+                    <max_acceleration>2.0</max_acceleration>
+                    <topic>${namespace}cmd_vel</topic>
+                    <odom_topic>${namespace}odom</odom_topic>
+                    <frame_id>${namespace}odom</frame_id>
+                    <child_frame_id>${namespace}base_footprint</child_frame_id>
+                    <odom_publisher_frequency>30</odom_publisher_frequency>
+                    <tf_topic>/tf</tf_topic>
+                </plugin>
+                <plugin filename="gz-sim-joint-state-publisher-system" name="gz::sim::systems::JointStatePublisher">
+                    <topic>${namespace}joint_states</topic>
+                    <joint_name>${namespace}l_wheel_joint</joint_name>
+                    <joint_name>${namespace}r_wheel_joint</joint_name>
+                </plugin>
+            </xacro:unless>
             <plugin filename="gz-sim-lamp-control-system" name="pinky_gz_sim::LampControlPlugin">
-                <link>robot_lamp</link>
+                <link>${namespace}robot_lamp</link>
             </plugin>
         </gazebo>
-        <gazebo reference="l_wheel">
+        <gazebo reference="${namespace}l_wheel">
             <self_collide>0</self_collide>
             <mu1>200</mu1>
@@ -23,5 +48,5 @@
             <!-- <minDepth>0.001</minDepth> -->
         </gazebo>
-        <gazebo reference="r_wheel">
+        <gazebo reference="${namespace}r_wheel">
             <self_collide>0</self_collide>
             <mu1>200</mu1>
@@ -31,5 +56,5 @@
             <!-- <minDepth>0.001</minDepth> -->
         </gazebo>
-        <gazebo reference="caster_wheel">
+        <gazebo reference="${namespace}caster_wheel">
             <self_collide>0</self_collide>
             <mu1>0.1</mu1>
@@ -39,11 +64,12 @@
             <!-- <minDepth>0.001</minDepth> -->
         </gazebo>
-        <gazebo reference="robot_lamp_mount_fixed_joint">
+        <gazebo reference="${namespace}robot_lamp_mount_fixed_joint">
             <disableFixedJointLumping>true</disableFixedJointLumping>
         </gazebo>
-        <gazebo reference="rplidar_link">
-            <sensor name='gpu_lidar' type='gpu_lidar'>
-                <topic>${namespace}/scan</topic>
+        <gazebo reference="${namespace}rplidar_link">
+            <sensor name='${namespace}gpu_lidar' type='gpu_lidar'>
+                <topic>${namespace}scan</topic>
                 <update_rate>10</update_rate>
+                <gz_frame_id>${namespace}rplidar_link</gz_frame_id>
                 <lidar>
                     <scan>
@@ -75,6 +101,6 @@
             </sensor>
         </gazebo>
-        <gazebo reference="front_camera_link">
-            <sensor name="camera" type="camera">
+        <gazebo reference="${namespace}front_camera_link">
+            <sensor name="${namespace}camera" type="camera">
                 <camera>
                     <horizontal_fov>1.1519</horizontal_fov>
@@ -91,14 +117,16 @@
                 <update_rate>30</update_rate>
                 <visualize>true</visualize>
-                <topic>camera/image_raw</topic>
+                <topic>${namespace}camera/image_raw</topic>
+                <gz_frame_id>${namespace}front_camera_link</gz_frame_id>
             </sensor>
         </gazebo>
-        <gazebo reference="imu_link">
-            <sensor name="imu" type="imu">
+        <gazebo reference="${namespace}imu_link">
+            <sensor name="${namespace}imu" type="imu">
                 <always_on>1</always_on>
                 <update_rate>100</update_rate>
                 <visualize>true</visualize>
-                <topic>imu_raw</topic>
+                <topic>${namespace}imu_raw</topic>
                 <enable_metrics>true</enable_metrics>
+                <gz_frame_id>${namespace}imu_link</gz_frame_id>
             </sensor>
         </gazebo>

File: pinky_description/urdf/robot.urdf.xacro (robot description, xacro)
@@ -7,4 +7,5 @@
     <xacro:arg name="cam_tilt_deg" default="8"/>
     <xacro:arg name="screen_tilt_deg" default="-25"/>
+    <xacro:arg name="ros2_control" default="false"/>
     <xacro:insert_robot namespace="$(arg namespace)"
                         is_sim="$(arg is_sim)"
